File: DragonATXProtoVDG.kicad_sch (KiCad schematic)
At the start: 67 parts, among them IC1 74LS273, IC2 MC6847, IC3 MC14053, J3 JTAG, Q1 MMBT4401, Q2 NPN, Q3 NPN, Q4 NPN, Q5 NPN, Q6 NPN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

Commit message: convert to use lhm1251
Parts:
- removed C11, C12, C13: 10uF, Capacitor_SMD:CP_Elec_4x5.4, symbol Device:C_Polarized_Small
- removed unit 2 of PL1
- removed Q1: MMBT4401, Library:SOT-23-3, symbol Simulation_SPICE:NPN
- removed Q2, Q3, Q4, Q5, Q6: NPN, Library:SOT-23-3, symbol Simulation_SPICE:NPN
- removed R10, R11, R12, R13: 150R, Resistor_SMD:R_0805_2012Metric_Pad1.20x1.40mm_HandSolder, symbol Device:R_Small
- removed R14: 3K3, Resistor_SMD:R_0805_2012Metric_Pad1.20x1.40mm_HandSolder, symbol Device:R_Small
- removed R15: 2K2, Resistor_SMD:R_0805_2012Metric_Pad1.20x1.40mm_HandSolder, symbol Device:R_Small
- removed R16, R20: 2K, Resistor_SMD:R_0805_2012Metric_Pad1.20x1.40mm_HandSolder, symbol Device:R_Small
- removed R17: 6K8, Resistor_SMD:R_0805_2012Metric_Pad1.20x1.40mm_HandSolder, symbol Device:R_Small
- removed R18: 4K7, Resistor_SMD:R_0805_2012Metric_Pad1.20x1.40mm_HandSolder, symbol Device:R_Small
- removed R19: 2K7, Resistor_SMD:R_0805_2012Metric_Pad1.20x1.40mm_HandSolder, symbol Device:R_Small
- removed R21, R22, R23: 150R, Resistor_SMD:R_0603_1608Metric, symbol Device:R_Small
- removed R7: 180R, Resistor_SMD:R_0805_2012Metric_Pad1.20x1.40mm_HandSolder, symbol Device:R_Small
- removed R8: 910R, Resistor_SMD:R_0805_2012Metric_Pad1.20x1.40mm_HandSolder, symbol Device:R_Small
- removed R9: 100R, Resistor_SMD:R_0805_2012Metric_Pad1.20x1.40mm_HandSolder, symbol Device:R_Small
- removed RV1, RV2, RV3: 50K, Potentiometer_SMD:Potentiometer_Bourns_TC33X_Vertical, symbol Device:R_Potentiometer_Trim
- added C14, C21: 10uF, Capacitor_SMD:CP_Elec_4x5.4, symbol Device:C_Polarized_Small
- added C20, C9: 0.1uF, Capacitor_SMD:C_0805_2012Metric_Pad1.18x1.45mm_HandSolder, symbol Device:C_Small
- added R27, R5: 10K, Resistor_SMD:R_0805_2012Metric_Pad1.20x1.40mm_HandSolder, symbol Device:R_Small
- added U2: LMH1251, Package_SO:TSSOP-24_4.4x7.8mm_P0.65mm, symbol Library:LMH1251
- C1, C10, C8: LCSC (none) -> C22387953
- C15, C5, C6: footprint Capacitor_Tantalum_SMD:CP_EIA-3216-12_Kemet-S -> Capacitor_Tantalum_SMD:CP_EIA-3528-21_Kemet-B; LCSC (none) -> C30242
- C16, C17, C18, C19, C3, C4, C7: LCSC (none) -> C28233
- C2: LCSC (none) -> C445063
- IC1: LCSC (none) -> C206102
- IC2: LCSC (none) -> C72123
- IC3: LCSC (none) -> C6742
- J3, TP1, TP2, TP3, TP4: now left out of the parts list
- PL1: footprint Library:Card_Edge -> Library:Card_Edge_Short; now left out of the parts list
- R1, R2, R3: LCSC (none) -> C141697
- R24: LCSC (none) -> C114556
- R25: LCSC (none) -> C114545
- R26: LCSC (none) -> C17398
- R4, R6: LCSC (none) -> C84376
- U1: now not fitted
- U3: value ATF1502ASL-xAx44 -> ATF1504ASL-xAx44; now not fitted
Connections:
- net +5V: now also Y2.4 (Vdd), C14.1, C20.1, C21.1, C9.2, R5.1, U2.17 (VCC), U2.7 (VCC)
- net BLUE: now also U2.18 (Bout)
- net GND: now also C14.2, C20.2, C21.2, C9.1, R27.1, U2.12 (GND), U2.16 (GND), U2.21 (Sleep), U2.22 (SD/HD), U2.23 (AUTO), U2.6 (GND); no longer Y2.4 (Vdd)
- net GREEN: now also U2.19 (Gout)
- net LUM': now also U2.10 (Y)
- net RED: now also U2.20 (Rout)
- net phiA: now also U2.8 (PRin)
- net phiB: now also U2.9 (PBin)
- new net: R27.2, U2.15 (Rext)
- new net: R5.2, U2.24 (Select)
- no-connect marks 56 -> 64
Other:
- moved on the sheet: C1, C10, C15, C2, C3, C4, C5, C6, C7, C8, IC1, IC2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

Commit message: condition rgb
Parts:
- added C11, C12, C13: 100uF, Capacitor_Tantalum_SMD:CP_EIA-2012-12_Kemet-R, symbol Device:C_Polarized_Small
- added D1, D2: SDM40E20LA, PCM_Package_TO_SOT_SMD_AKL:SOT-23, symbol PCM_Diode_Schottky_AKL:SDM40E20LA
- added R10, R11, R12: 33R, Resistor_SMD:R_0805_2012Metric_Pad1.20x1.40mm_HandSolder, symbol Device:R_Small
- added R7, R8, R9: 10K, Resistor_SMD:R_0805_2012Metric_Pad1.20x1.40mm_HandSolder, symbol Device:R_Small
- U1, U2: now fitted
Connections:
- net BLUE: now also C13.2, D2.2 (K2), R12.1, R9.2; no longer U1.8 (BLUE), U2.18 (Bout)
- net GND: now also D1.3 (A), D2.3 (A), R7.1, R8.1, R9.1
- net GREEN: now also C12.2, D1.1 (K1), R11.1, R8.2; no longer U1.7 (GREEN), U2.19 (Gout)
- net RED: now also C11.2, D1.2 (K2), R10.1, R7.2; no longer U1.6 (RED), U2.20 (Rout)
- new net: R12.2, U1.8 (BLUE)
- new net: C12.1, U2.19 (Gout)
- new net: C11.1, U2.20 (Rout)
- new net: R10.2, U1.6 (RED)
- new net: R11.2, U1.7 (GREEN)
- new net: C13.1, U2.18 (Bout)
- no-connect marks 64 -> 65
Other:
- moved on the sheet: C14, C20, C21, C9, R27, R5
